File: hardware/UPP_simple/UPP_simple.kicad_sch (KiCad schematic)
At the start: 0 parts

Commit message: Add files via upload
Parts:
- added C9: 330n, symbol Device:C
- added IC2: STM32G0C1KCT6N, QFP80P900X900X160-32N, symbol STM32G0C1KCT6N:STM32G0C1KCT6N
- added R10, R11, R12, R13, R14, R15, R9: 47R, symbol Device:R
Connections:
- new net: IC2.14 (PA7), R9.1
- new net: IC2.15 (PB0), R12.1
- new net: IC2.12 (PA5), R11.1
- new net: IC2.10 (PA3), R13.1
- new net: IC2.9 (PA2), R14.1
- new net: IC2.13 (PA6), R10.1
- new net: IC2.16 (PB1), R15.1
- new net 3V3: C9.1, IC2.4 (VDD/VDDA)
- new net ADC.CLK: R11.2
- new net ADC.CS: R13.2
- new net ADC.DRDY: R12.2
- new net ADC.MISO: R10.2
- new net ADC.MOSI: R9.2
- new net ADC.RST: R15.2
- new net ADC.START: R14.2
- new net GND: C9.2, IC2.5 (VSS/VSSA)
- no-connect marks 0 -> 1
Other:
- removed sheet adc
- removed sheet power
- added sheet ADC (adc.kicad_sch)
- added sheet Power (power.kicad_sch)
- company: (none) -> Author: Kacper Pawlak
- title: (none) -> Universal use measuring PCB
