File: hardware/UPP_simple/adc.kicad_sch (KiCad schematic)
At the start: 12 parts, among them IC1 ADS114S08BIPBSR, IC2 STM32G0C1KCT6N

Commit message: Add files via upload
Parts:
- removed C9: 330n, symbol Device:C
- removed IC2: STM32G0C1KCT6N, QFP80P900X900X160-32N, symbol STM32G0C1KCT6N:STM32G0C1KCT6N
- removed R10, R11, R12, R13, R14, R15, R9: 47R, symbol Device:R
Connections:
- net GND: now also IC1.14 (DGND)
- net ADC_START renamed ADC.START
- net DRDY renamed ADC.DRDY
- net RST renamed ADC.RST
- net SPI_CLK renamed ADC.CLK
- net SPI_CS renamed ADC.CS
- net SPI_MISO renamed ADC.MISO
- net SPI_MOSI renamed ADC.MOSI
Other:
- company: (none) -> Author: Kacper Pawlak
- title: (none) -> Universal use measuring PCB
- moved on the sheet: C1, C2, IC1
