File: hardware/UPP_simple/adc.kicad_sch (KiCad schematic)
At the start: 3 parts, among them IC1 ADS114S08BIPBSR

Commit message: Add files via upload
Parts:
- removed C1: 330n, Capacitor_SMD:C_0603_1608Metric_Pad1.08x0.95mm_HandSolder, symbol Device:C
- added C1, C3: 100n, symbol Device:C_Small
- C2: value 330n -> 1u
Connections:
- net +5V: now also C1.2
- net GND: now also IC1.24 (REFCOM), IC1.27 (AVSS_1), IC1.28 (AVSS_2), C1.1, C3.2; no longer IC1.23 (REFOUT)
- net 3V3: now reaches IC1.15 (IOVDD)
- net 3V3: now also IC1.16 (DVDD), C3.1
- net at C2.1: now also IC1.23 (REFOUT); no longer IC1.24 (REFCOM)
- net ADC_SPI.CS renamed ADC_SPI.NSS
- no-connect marks 5 -> 3
Other:
- moved on the sheet: C2, IC1
