File: hardware/UPP_simple/analog_inputs.kicad_sch (KiCad schematic)
At the start: 98 parts, among them J1 Conn_01x03, J10 Conn_01x04, J11 Conn_01x04, J19 Conn_01x04, J2 Conn_01x03, J3 Conn_01x03, J4 Conn_01x03, J5 Conn_01x03, J6 Conn_01x03, J7 Conn_01x04, J8 Conn_01x04, J9 Conn_01x04, U1 Opamp_Quad, U2 Opamp_Quad, U3 Opamp_Quad

Commit message: Add files via upload
Parts:
- removed J19: Conn_01x04, symbol Connector_Generic:Conn_01x04
- removed JP1, JP10, JP11, JP12, JP13, JP14, JP15, JP16, JP17, JP18, JP19, JP2, JP20, JP21, JP22, JP23, JP24, JP4, JP5, JP6, JP7, JP8, JP9: Jumper_3_Open, symbol Jumper:Jumper_3_Open
- removed unit 5 of U2
- removed unit 5 of U3
- added C11, C12, C9: 100n, Capacitor_SMD:C_0603_1608Metric, symbol Device:C_Small
- added J14: Conn_01x04, symbol Connector_Generic:Conn_01x04
- added JP1, JP10, JP11, JP13, JP14, JP15, JP16, JP17, JP18, JP19, JP2, JP20, JP21, JP22, JP23, JP24, JP25, JP26, JP3, JP31, JP32, JP33, JP34, JP35, JP36, JP37, JP38, JP39, JP4, JP40, JP41, JP42, JP43, JP44, JP45, JP46, JP47, JP5, JP6, JP7, JP8, JP9: SolderJumper_3_Bridged12, Jumper:SolderJumper-3_P1.3mm_Bridged12_Pad1.0x1.5mm, symbol Jumper:SolderJumper_3_Bridged12
- added R64, R66, R67, R68, R69, R71, R72, R74, R75, R76, R77, R79, R80: 10k, Resistor_SMD:R_0603_1608Metric_Pad0.98x0.95mm_HandSolder, symbol Device:R_Small
- added R65, R73, R81: 5k, Resistor_SMD:R_0603_1608Metric_Pad0.98x0.95mm_HandSolder, symbol Device:R_Small
- added R70, R78: 12k, Resistor_SMD:R_0603_1608Metric_Pad0.98x0.95mm_HandSolder, symbol Device:R_Small
- added U6, U7: Opamp_Quad, symbol Device:Opamp_Quad
- R29, R38: value 3k92 -> 12k
- R30, R35, R40, R51, R53, R55: value 20k5 -> 10k
- R31, R47, R48: value 3k92 -> 10k
- R32: value 1k -> 5k
- R34, R39, R50, R52: value 1k -> 10k
- R41: value 10k -> 5k
- R46: value 10k -> 12k
- R49: value 3k92 -> 5k
- R54: value 1k -> 12k
- U1, U2, U3: footprint (none) -> Footprints:SOP65P640X120-14N
Connections:
- net +12V: now also JP1.3 (B), JP10.3 (B), JP11.3 (B), JP13.3 (B), JP18.3 (B), JP2.3 (B), JP23.3 (B), JP26.3 (B), JP33.3 (B), JP38.3 (B), JP43.3 (B), JP9.3 (B)
- net +5V: now also C11.1, C12.1, C9.1, JP1.1 (A), JP10.1 (A), JP11.1 (A), JP13.1 (A), JP18.1 (A), JP2.1 (A), JP23.1 (A), JP26.1 (A), JP33.1 (A), JP38.1 (A), JP43.1 (A), JP9.1 (A), U6.4 (V+), U7.4 (V+)
- net DIF1: now also R31.2
- net DIF2: now also R40.2, R41.2; no longer R34.2
- net DIF3: now also R48.2, R49.2; no longer R39.2
- net DIF4: now also R64.2, R65.2; no longer R50.2
- net DIF5: now also R72.2, R73.2; no longer R52.2
- net DIF6: now also R80.2, R81.2; no longer R54.2
- net GND: now also R29.2, R38.2, R39.2, R46.2, R47.2, R54.2, C11.2, C12.2, C9.2, J14.1 (Pin_1), R70.2, R71.2, R78.2, R79.2, U6.11 (V-), U7.11 (V-); no longer R29.1, R31.1, R35.2, R38.1, R40.2, R47.1, R48.1, R49.1, R51.2, R53.2
- net at J9.4 (Pin_4): now also JP23.2 (C)
- net at R1.1: now also JP3.1 (A)
- net at J11.2 (Pin_2): now also JP40.2 (C); no longer R46.1
- net at R45.1: now also JP25.3 (B); no longer J11.3 (Pin_3)
- net at J11.4 (Pin_4): now also JP38.2 (C)
- net at R53.1: now also JP35.3 (B)
- net at J7.2 (Pin_2): now also JP15.2 (C); no longer R27.1
- net at J7.3 (Pin_3): now also JP14.2 (C); no longer R26.1
- net at J7.4 (Pin_4): now also JP13.2 (C)
- net at R8.2, U2.9 (-): now also R26.2, JP16.2 (C); no longer R32.1
- net at R28.1: now also JP15.3 (B)
- net at R28.2, U2.10 (+): now also R27.2, JP17.2 (C)
- net at J4.3 (Pin_3): now also JP2.2 (C)
- net at R17.2: now also JP4.3 (B)
- net at J4.2 (Pin_2): now also JP4.2 (C)
- net at R33.1: now also JP4.1 (A)
- net at R21.2: now also JP7.3 (B)
- net at J5.2 (Pin_2): now also JP7.2 (C)
- net at R20.1: now also JP7.1 (A)
- net at J3.3 (Pin_3): now also JP9.2 (C)
- net at R16.2: now also JP8.3 (B)
- net at R30.1: now also JP17.1 (A)
- net at J5.3 (Pin_3): now also JP10.2 (C)
- net at R7.1: now also JP8.1 (A)
- net at J1.2 (Pin_2): now also JP3.2 (C)
- net at J1.3 (Pin_3): now also JP1.2 (C)
- net at R36.1: now also JP20.1 (A); no longer J8.3 (Pin_3)
- net at J8.2 (Pin_2): now also JP20.2 (C); no longer R37.1
- net at U3.3 (+): now also R44.2, R45.2, JP32.2 (C); no longer R37.2
- net at R55.1: now also JP37.1 (A)
- net at R2.2: now also JP3.3 (B)
- net at U3.5 (+): now also JP47.2 (C), R76.2, R77.2; no longer R46.2
- net at R44.1: now also JP25.1 (A); no longer J10.2 (Pin_2)
- net at J10.3 (Pin_3): now also JP34.2 (C); no longer R43.1
- net at J10.4 (Pin_4): now also JP33.2 (C)
- net at U3.10 (+): now also JP42.2 (C), R68.2, R69.2; no longer R44.2
- net at R35.1: now also JP19.3 (B)
- net at J6.3 (Pin_3): now also JP11.2 (C)
- net at J6.2 (Pin_2): now also JP6.2 (C)
- net at R4.1: now also JP5.1 (A)
- net at R8.1: now also JP14.1 (A)
- net at J8.4 (Pin_4): now also JP18.2 (C)
- net at R40.1: now also JP21.1 (A)
- net at J9.2 (Pin_2): now also JP25.2 (C); no longer R42.1
- net at R42.2: now also R43.2, U3.2 (-), JP31.2 (C); no longer U3.12 (+)
- net at J9.3 (Pin_3): now also JP24.2 (C); no longer R41.1
- net at R23.1: now also JP6.1 (A)
- net at J2.3 (Pin_3): now also JP26.2 (C)
- net at R51.1: now also JP34.3 (B)
- net at U2.12 (+): now also R36.2, R37.2, JP22.2 (C); no longer R27.2
- net at R5.2: now also JP5.3 (B)
- net at R24.2: now also JP6.3 (B)
- net at J3.2 (Pin_2): now also JP8.2 (C)
- net at J2.2 (Pin_2): now also JP5.2 (C)
- new net: JP31.1 (A), R48.1
- new net: JP31.3 (B), R49.1
- new net: JP32.1 (A), R47.1
- new net: JP41.1 (A), R72.1
- new net: JP37.3 (B), R54.1
- new net: JP36.1 (A), R64.1
- new net: JP40.1 (A), R68.1
- new net: JP40.3 (B), R69.1
- new net: JP41.2 (C), R66.2, R67.2, U3.9 (-)
- new net: JP41.3 (B), R73.1
- new net: JP47.1 (A), R79.1
- new net: JP47.3 (B), R78.1
- new net: JP22.1 (A), R39.1
- new net: JP22.3 (B), R38.1
- new net: JP20.3 (B), R37.1
- new net: JP46.3 (B), R81.1
- new net: JP16.3 (B), R32.1
- new net: JP36.3 (B), R65.1
- new net: JP45.1 (A), R76.1
- new net: J14.2 (Pin_2), JP45.2 (C)
- new net: JP45.3 (B), R77.1
- new net: JP19.1 (A), R34.1
- new net: J8.3 (Pin_3), JP19.2 (C)
- new net: JP36.2 (C), R50.2, R51.2, U3.13 (-)
- new net: JP14.3 (B), R26.1
- new net: JP21.2 (C), R34.2, R35.2, U2.13 (-)
- new net: JP16.1 (A), R31.1
- new net: JP44.1 (A), R74.1
- new net: J14.3 (Pin_3), JP44.2 (C)
- new net: JP44.3 (B), R75.1
- new net: JP37.2 (C), R52.2, R53.2, U3.12 (+)
- new net: J11.3 (Pin_3), JP39.2 (C)
- new net: JP46.2 (C), R74.2, R75.2, U3.6 (-)
- new net: JP35.1 (A), R52.1
- new net: JP42.1 (A), R71.1
- new net: JP42.3 (B), R70.1
- new net: JP39.1 (A), R66.1
- new net: JP39.3 (B), R67.1
- new net: JP17.3 (B), R29.1
- new net: J10.2 (Pin_2), JP35.2 (C)
- new net: JP34.1 (A), R50.1
- new net: JP15.1 (A), R27.1
- new net: JP32.3 (B), R46.1
- new net: JP21.3 (B), R41.1
- new net: JP46.1 (A), R80.1
- new net: JP24.1 (A), R42.1
- new net: JP24.3 (B), R43.1
- new net: J14.4 (Pin_4), JP43.2 (C)
- no-connect marks 1 -> 0
Other:
- moved on the sheet: U1E
