File: hardware/UMB/UMB.kicad_sch (KiCad schematic)
At the start: 0 parts

Commit message: All done except power
Other:
- sheet adc renamed ADC
- sheet analog renamed Analog
- sheet can renamed CAN
- sheet control renamed MCU
- sheet inputs renamed Connectors
- sheet power renamed Power
- sheet ADC: file adc.kicad_sch -> ADC.kicad_sch
- sheet Analog: file analog.kicad_sch -> Analog.kicad_sch
- sheet Analog ports: added {DIF1}, {DIF2}, {DIF3}, {DIF4}, {DIF5}, {DIF6}; removed none
- sheet CAN: file can.kicad_sch -> CAN.kicad_sch
- sheet CAN ports: added GND_CAN_ISO, {CAN}; removed none
- sheet Connectors: file inputs.kicad_sch -> Inputs.kicad_sch
- sheet Connectors ports: added GND_CAN_ISO, UART_RX, UART_TX, {CAN}, {DIF1}, {DIF2}, {DIF3}, {DIF4}, {DIF5}, {DIF6}, {ST-LINK}; removed none
- sheet MCU: file control.kicad_sch -> MCU.kicad_sch
- sheet MCU ports: added UART_RX, UART_TX, {ST-LINK}; removed none
- sheet Power: file power.kicad_sch -> Power.kicad_sch
