File: hardware/UMB/Analog.kicad_sch (KiCad schematic)
At the start: 54 parts, among them IC1 INA2128UA_1K, IC2 INA2128UA_1K, IC3 INA2128UA_1K, U7 TLC274AIDR, U8 TLC274AIDR, U9 TLC274AIDR

Commit message: All done except power
Parts:
- renumbered IC3 to U, IC2 to U, IC1 to U
Connections:
- net +12VA is gone; now on net +12V: C22.1, C23.1, C24.1, U.9 (V+), U.9 (V+), U.9 (V+)
- net +5VA is gone; now on net +5V: C25.1, C26.1, C27.1, U7.4 (V+), U8.4 (V+), U9.4 (V+)
- net DIF1_N renamed DIF1-
- net DIF1_P renamed DIF1+
- net DIF2_N renamed DIF2-
- net DIF2_P renamed DIF2+
- net DIF3_N renamed DIF3-
- net DIF3_P renamed DIF3+
- net DIF4_N renamed DIF4-
- net DIF4_P renamed DIF4+
- net DIF5_N renamed DIF5-
- net DIF5_P renamed DIF5+
- net DIF6_N renamed DIF6-
- net DIF6_P renamed DIF6+
Other:
- moved on the sheet: C22, C23, C24, C25, C26, C27, D10, D11, D12, D6, D8, D9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

Commit message: Power section done
Parts:
- removed C22, C23, C24: 100n, Capacitor_SMD:C_0603_1608Metric, symbol Device:C_Small
- removed D10, D11, D12, D6, D8, D9: ESD9B5.0ST5G, Diode_SMD:D_SOD-923, symbol Diode:ESD9B5.0ST5G
- removed JP13, JP14, JP15, JP16, JP17, JP18, JP19, JP20, JP21, JP22, JP23, JP24: Jumper_3_Bridged12, Connector_PinHeader_1.00mm:PinHeader_1x03_P1.00mm_Vertical, symbol Jumper:Jumper_3_Bridged12
- removed R27: 14k, Resistor_SMD:R_0603_1608Metric_Pad0.98x0.95mm_HandSolder, symbol Device:R_Small
- removed U (x3): INA2128UA_1K, SOIC127P1030X265-16N, symbol INA2128UA_1K:INA2128UA_1K
- removed U7, U8, U9: TLC274AIDR, SOIC127P600X175-14N, symbol Device:Opamp_Quad
- added C35, C36, C40: 100n, Capacitor_SMD:C_0603_1608Metric_Pad1.08x0.95mm_HandSolder, symbol Device:C_Small
- added J1, J2, J3, J4, J5, J6: PinHeader 02x04, Connector_PinHeader_1.00mm:PinHeader_2x04_P1.00mm_Vertical, symbol Connector_Generic:Conn_02x04_Counter_Clockwise
- added JP1, JP2, JP3, JP4, JP5, JP6: PH1-03-UA, Connector_PinHeader_1.00mm:PinHeader_1x03_P1.00mm_Vertical, symbol Jumper:Jumper_3_Bridged12
- added R14, R50: 14k, Resistor_SMD:R_0603_1608Metric_Pad0.98x0.95mm_HandSolder, symbol Device:R_Small
- added R15, R21, R49: 12.4k, Resistor_SMD:R_0603_1608Metric_Pad0.98x0.95mm_HandSolder, symbol Device:R_Small
- added R16, R23, R30, R51: 2.1k, Resistor_SMD:R_0603_1608Metric_Pad0.98x0.95mm_HandSolder, symbol Device:R_Small
- added R17, R24, R31, R45, R52: 499R, Resistor_SMD:R_0603_1608Metric_Pad0.98x0.95mm_HandSolder, symbol Device:R_Small
- added R18, R32, R46, R54: 0R, Resistor_SMD:R_0603_1608Metric_Pad0.98x0.95mm_HandSolder, symbol Device:R_Small
- added R19, R25, R47, R53: 49.9R, Resistor_SMD:R_0603_1608Metric_Pad0.98x0.95mm_HandSolder, symbol Device:R_Small
- added R20, R48, R55: 10k, Resistor_SMD:R_0603_1608Metric_Pad0.98x0.95mm_HandSolder, symbol Device:R_Small
- added U11, U13, U14: TLC274AIDR, SOIC-14:SOIC127P600X175-14N, symbol TLC274AIDR:TLC274AIDR
- added U12, U15, U16: INA2128UA_1K, SOIC127P1030X265-16N, symbol INA2128UA_1K:INA2128UA_1K
- C37: renamed from C25; footprint Capacitor_SMD:C_0603_1608Metric -> Capacitor_SMD:C_0603_1608Metric_Pad1.08x0.95mm_HandSolder; Mouser (none) -> https://www.mouser.pl/ProductDetail/KEMET/C0603C104M4RACAUT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; Mouser No (none) -> 80-C0603C104M4RAUTO
- C38: renamed from C26; footprint Capacitor_SMD:C_0603_1608Metric -> Capacitor_SMD:C_0603_1608Metric_Pad1.08x0.95mm_HandSolder; Mouser (none) -> https://www.mouser.pl/ProductDetail/KEMET/C0603C104M4RACAUT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; Mouser No (none) -> 80-C0603C104M4RAUTO
- C39: renamed from C27; footprint Capacitor_SMD:C_0603_1608Metric -> Capacitor_SMD:C_0603_1608Metric_Pad1.08x0.95mm_HandSolder; Mouser (none) -> https://www.mouser.pl/ProductDetail/KEMET/C0603C104M4RACAUT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; Mouser No (none) -> 80-C0603C104M4RAUTO
- R28: value 0R -> 14k
- R29, R35: value 10k -> 12.4k
- R33, R39: value 14k -> 49.9R
- R34: value 0R -> 10k
- R37: value 0R -> 2.1k
- R38: value 10k -> 499R
- R43: value 0R -> 12.4k
- R44: value 10k -> 2.1k
- renumbered D7 to D2, D2 to D3, D1 to D5, D3 to D6, D5 to D7, R30 to R22, R31 to R26, R32 to R27
Connections:
- net +5V: now also U11.4 (V+), U13.4 (V+), U14.4 (V+)
- net AGND: now also R27.2, R34.2, R41.2, C35.1, C36.1, C40.1, R20.2, R48.2, R55.2, U11.11 (V-), U12.12 (REFB), U12.5 (REFA), U12.8 (V-), U13.11 (V-), U14.11 (V-), U15.12 (REFB), U15.5 (REFA), U15.8 (V-), U16.12 (REFB), U16.5 (REFA), U16.8 (V-); no longer R27.1, R29.1, R35.1, R38.1, R41.1, R44.1
- net DIF1: now also U11.10 (+), U11.8
- net DIF1+: now also U12.2 (V+INA)
- net DIF1-: now also U12.1 (V-INA)
- net DIF1_12: now also JP1.2 (C), U12.6 (VOA), U12.7 (SENSEA)
- net DIF2: now also U11.12 (+), U11.14
- net DIF2+: now also U12.15 (V+INB)
- net DIF2-: now also U12.16 (V-INB)
- net DIF2_12: now also JP2.2 (C), U12.10 (SENSEB), U12.11 (VOB)
- net DIF3: now also U14.1, U14.3 (+)
- net DIF3+: now also U15.2 (V+INA)
- net DIF3-: now also U15.1 (V-INA)
- net DIF3_12: now also JP3.2 (C), U15.6 (VOA), U15.7 (SENSEA)
- net DIF4: now also U14.5 (+), U14.7
- net DIF4+: now also U15.15 (V+INB)
- net DIF4-: now also U15.16 (V-INB)
- net DIF4_12: now also JP4.2 (C), U15.10 (SENSEB), U15.11 (VOB)
- net DIF5: now also U14.10 (+), U14.8
- net DIF5+: now also U16.2 (V+INA)
- net DIF5-: now also U16.1 (V-INA)
- net DIF5_12: now also JP5.2 (C), U16.6 (VOA), U16.7 (SENSEA)
- net DIF6: now also U14.12 (+), U14.14
- net DIF6+: now also U16.15 (V+INB)
- net DIF6-: now also U16.16 (V-INB)
- net DIF6_12: now also JP6.2 (C), U16.10 (SENSEB), U16.11 (VOB)
- net SE1: now also U13.1, U13.3 (+)
- net SE2: now also U13.5 (+), U13.7
- net SE3: now also U13.10 (+), U13.8
- net SE4: now also U13.12 (+), U13.14
- net SE5: now also U11.1, U11.3 (+)
- net SE6: now also U11.5 (+), U11.7
- net at R28.1: now also R34.1, R32.2, U14.2 (-)
- net at R28.2: now also JP3.1 (A); no longer R29.2
- net RGA5_1: now reaches R43.2, R44.2
- net RGA5_1: now also R45.2, R47.2, U16.3 (RGA_1); no longer R42.1
- net at R22.1, R26.2: now also R27.1, U11.13 (-); no longer R27.2
- net RGA4_1: now reaches R37.2, R38.2
- net RGA4_1: now also R35.2, R39.2, U15.14 (RGB_2); no longer R36.1
- net at R22.2: now also JP2.1 (A)
- net at R37.1: now also J4.2 (Pin_2)
- net RGA3_1: now reaches R33.2
- net RGA3_1: now also R29.2, R30.2, R31.2, U15.3 (RGA_1)
- net at R40.1: now also JP4.3 (B)
- net at R42.2: now also JP5.1 (A)
- net at R26.1: now also JP2.3 (B)
- net at R43.1: now also J5.1 (Pin_1)
- net at R36.2: now also JP4.1 (A)
- new net: J3.1 (Pin_1), R29.1
- new net: J2.4 (Pin_4), R25.1
- new net: J5.4 (Pin_4), R47.1
- new net: R36.1, R40.2, R41.1, U14.6 (-)
- new net: J6.4 (Pin_4), R53.1
- new net: R50.1, R54.2, R55.1, U14.13 (-)
- new net: JP6.1 (A), R50.2
- new net: J5.2 (Pin_2), R44.1
- new net: J5.3 (Pin_3), R45.1
- new net: J3.3 (Pin_3), R31.1
- new net: J6.3 (Pin_3), R52.1
- new net: J3.2 (Pin_2), R30.1
- new net: J3.4 (Pin_4), R33.1
- new net: JP3.3 (B), R32.1
- new net: JP1.3 (B), R18.1
- new net: R14.1, R18.2, R20.1, U11.9 (-)
- new net: R42.1, R46.2, R48.1, U14.9 (-)
- new net: J6.1 (Pin_1), R49.1
- new net: J6.2 (Pin_2), R51.1
- new net: J1.4 (Pin_4), R19.1
- new net: J4.1 (Pin_1), R35.1
- new net: J1.1 (Pin_1), R15.1
- new net: J4.3 (Pin_3), R38.1
- new net: J4.4 (Pin_4), R39.1
- new net: J2.3 (Pin_3), R24.1
- new net: JP1.1 (A), R14.2
- new net: JP6.3 (B), R54.1
- new net: J2.1 (Pin_1), R21.1
- new net: J2.2 (Pin_2), R23.1
- new net: JP5.3 (B), R46.1
- new net: J1.3 (Pin_3), R17.1
- new net: J1.2 (Pin_2), R16.1
- new net +12VA: C35.2, C36.2, C40.2, U12.9 (V+), U15.9 (V+), U16.9 (V+)
- new net RGA1_1: R15.2, R16.2, R17.2, R19.2, U12.3 (RGA_1)
- new net RGA1_2: J1.5 (Pin_5), J1.6 (Pin_6), J1.7 (Pin_7), J1.8 (Pin_8), U12.4 (RGA_2)
- new net RGA2_1: R21.2, R23.2, R24.2, R25.2, U12.14 (RGB_2)
- new net RGA2_2: J2.5 (Pin_5), J2.6 (Pin_6), J2.7 (Pin_7), J2.8 (Pin_8), U12.13 (RGB_1)
- new net RGA3_2: J3.5 (Pin_5), J3.6 (Pin_6), J3.7 (Pin_7), J3.8 (Pin_8), U15.4 (RGA_2)
- new net RGA4_2: J4.5 (Pin_5), J4.6 (Pin_6), J4.7 (Pin_7), J4.8 (Pin_8), U15.13 (RGB_1)
- new net RGA5_2: J5.5 (Pin_5), J5.6 (Pin_6), J5.7 (Pin_7), J5.8 (Pin_8), U16.4 (RGA_2)
- new net RGA6_1: R49.2, R51.2, R52.2, R53.2, U16.14 (RGB_2)
- new net RGA6_2: J6.5 (Pin_5), J6.6 (Pin_6), J6.7 (Pin_7), J6.8 (Pin_8), U16.13 (RGB_1)
- new net SE1IN: U13.2 (-)
- new net SE2IN: U13.6 (-)
- new net SE3IN: U13.9 (-)
- new net SE4IN: U13.13 (-)
- new net SE5IN: U11.2 (-)
- new net SE6IN: U11.6 (-)
- no-connect marks 12 -> 0
Other:
- note added: "ADC is 5V analog"
- note added: "Setting gain: G = 1 + 50k/R NC - 1 12.4k - 5 2.1k - 25 499R - 100 49.9R - 1000"
- moved on the sheet: C37, C38, C39, D2, D3, D4, D5, D6, D7, R22, R26, R27

Commit message: Added all footprints and parts Mouser IDs
Parts:
- C35, C36, C37, C38, C39, C40: Manufacturer_Part_Number (none) -> C0603C104M4RACAUTO
- D2, D3, D4, D5, D6, D7: Manufacturer_Part_Number (none) -> ESD9B5.0ST5G; Mouser (none) -> https://www.mouser.pl/ProductDetail/onsemi/ESD9B5.0ST5G?qs=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; Mouser No (none) -> 863-ESD9B5.0ST5G
- J1, J2, J3, J4, J5, J6: Header https://www.mouser.pl/ProductDetail/Adam-Tech/PH2-04-UA?qs=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 -> (none); Manufacturer_Part_Number (none) -> PH2-04-UA; Mouser (none) -> https://www.mouser.pl/ProductDetail/Adam-Tech/PH2-04-UA?qs=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; Mouser No (none) -> 737-PH2-04-UA
- JP1, JP2, JP3, JP4, JP5, JP6: Header https://www.mouser.pl/ProductDetail/Adam-Tech/PH1-03-UA?qs=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 -> (none); Jumper https://botland.com.pl/zworki/556-zworka-jumper-10szt-59044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 -> (none)
- R14, R22, R28, R36, R42, R50: Manufacturer_Part_Number (none) -> RT0603DRD0714KL; Mouser (none) -> https://www.mouser.pl/ProductDetail/YAGEO/RT0603DRD0714KL?q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; Mouser No (none) -> 603-RT0603DRD0714KL
- R15, R21, R29, R35, R43, R49: Manufacturer_Part_Number (none) -> RT0603BRD0712K4L; Mouser (none) -> https://www.mouser.pl/ProductDetail/YAGEO/RT0603BRD0712K4L?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; Mouser No (none) -> 603-RT0603BRD0712K4L
- R16, R23, R30, R37, R44, R51: Manufacturer_Part_Number (none) -> RT0603BRD072K1L; Mouser (none) -> https://www.mouser.pl/ProductDetail/YAGEO/RT0603BRD072K1L?q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; Mouser No (none) -> 603-RT0603BRD072K1L
- R17, R24, R31, R38, R45, R52: Manufacturer_Part_Number (none) -> ERA-3AEB4990V; Mouser (none) -> https://www.mouser.pl/ProductDetail/Panasonic/ERA-3AEB4990V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; Mouser No (none) -> 667-ERA-3AEB4990V
- R18, R20, R26, R27, R32, R34, R40, R41, R46, R48, R54, R55: Mouser (none) -> in warszatowe zapasy i think
- R19, R25, R33, R39, R47, R53: Manufacturer_Part_Number (none) -> ERA-3AEB49R9V; Mouser (none) -> https://www.mouser.pl/ProductDetail/Panasonic/ERA-3AEB49R9V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; Mouser No (none) -> 667-ERA-3AEB49R9V
- U11, U13, U14: Height 1.75 -> (none); Manufacturer_Name Texas Instruments -> (none); Mouser (none) -> https://www.mouser.pl/ProductDetail/Texas-Instruments/TLC27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; Mouser No (none) -> 595-TLC274AIDR; Mouser Part Number 595-TLC274AIDR -> (none); Mouser Price/Stock https://www.mouser.co.uk/ProductDetail/Texas-Instruments/TL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 -> (none)
- U12, U15, U16: Height 2.65 -> (none); Manufacturer_Name Texas Instruments -> (none); Manufacturer_Part_Number INA2128UA/1K -> INA2128UA; Mouser (none) -> https://www.mouser.pl/ProductDetail/Texas-Instruments/INA21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; Mouser No (none) -> 595-INA2128UA/1K; Mouser Part Number 595-INA2128UA/1K -> (none); Mouser Price/Stock https://www.mouser.co.uk/ProductDetail/Texas-Instruments/IN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 -> (none)
