File: hardware/UMB/MCU.kicad_sch (KiCad schematic)
At the start: 9 parts, among them U1 STM32G0C1KCTxN

Commit message: Power section done
Parts:
- C1: footprint (none) -> Capacitor_SMD:C_0603_1608Metric_Pad1.08x0.95mm_HandSolder; Mouser (none) -> https://www.mouser.pl/ProductDetail/KEMET/C0603C104M4RACAUT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; Mouser No (none) -> 80-C0603C104M4RAUTO
- renumbered R4 to R1, R5 to R2, R6 to R3, R1 to R4, R7 to R5, R2 to R6, R3 to R7
Connections:
- net +3.3V: now also C1.1; no longer C1.2
- net GND: now also C1.2; no longer C1.1
- no-connect marks 13 -> 14

Commit message: Added all footprints and parts Mouser IDs
Parts:
- C1: Manufacturer_Part_Number (none) -> C0603C104M4RACAUTO
- R1, R2, R3, R4, R5, R6, R7: Manufacturer_Part_Number (none) -> RT0603DRD0747RL; Mouser (none) -> https://www.mouser.pl/ProductDetail/YAGEO/RT0603DRD0747RL?q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; Mouser No (none) -> 603-RT0603DRD0747RL
- U1: Manufacturer_Part_Number (none) -> STM32G0C1KCT6N; Mouser (none) -> https://www.mouser.pl/ProductDetail/STMicroelectronics/STM3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; Mouser No (none) -> 511-STM32G0C1KCT6N
Changed lines of the file:
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@@
 			)
 		)
-		(property "Datasheet" "~"
+		(property "Datasheet" "https://www.mouser.pl/datasheet/3/508/1/PYu-RT_1-to-0.01_RoHS_L_15.pdf"
 			(at 96.52 110.49 0)
 			(effects
@@
 			)
 		)
-		(property "Sim.Device" ""
+		(property "Manufacturer_Part_Number" "RT0603DRD0747RL"
 			(at 96.52 110.49 90)
 			(effects
@@
 			)
 		)
-		(property "Sim.Library" ""
+		(property "Mouser" "https://www.mouser.pl/ProductDetail/YAGEO/RT0603DRD0747RL?qs=sGAEpiMZZMvdGkrng054t%252BSYh%252B1gqt95bcSQVS5MnP8%3D"
 			(at 96.52 110.49 90)
 			(effects
@@
 			)
 		)
-		(property "Sim.Name" ""
-			(at 96.52 110.49 90)
-			(effects
-				(font
-					(size 1.27 1.27)
-				)
-				(hide yes)
-			)
-		)
-		(property "Sim.Pins" ""
+		(property "Mouser No" "603-RT0603DRD0747RL"
 			(at 96.52 110.49 90)
 			(effects
@@
 		)
 		(property "Mouser" "https://www.mouser.pl/ProductDetail/KEMET/C0603C104M4RACAUTO?qs=sSYV1F9c5cFMyVgVMlPozw%3D%3D"
+			(at 129.54 59.69 0)
+			(effects
+				(font
+					(size 1.27 1.27)
+				)
+				(hide yes)
+			)
+		)
+		(property "Manufacturer_Part_Number" "C0603C104M4RACAUTO"
 			(at 129.54 59.69 0)
 			(effects
@@
 			)
 		)
-		(property "Datasheet" "~"
+		(property "Datasheet" "https://www.mouser.pl/datasheet/3/508/1/PYu-RT_1-to-0.01_RoHS_L_15.pdf"
 			(at 96.52 90.17 0)
 			(effects
@@
 			)
 		)
-		(property "Sim.Device" ""
+		(property "Manufacturer_Part_Number" "RT0603DRD0747RL"
 			(at 96.52 90.17 90)
 			(effects
@@
 			)
 		)
-		(property "Sim.Library" ""
+		(property "Mouser" "https://www.mouser.pl/ProductDetail/YAGEO/RT0603DRD0747RL?qs=sGAEpiMZZMvdGkrng054t%252BSYh%252B1gqt95bcSQVS5MnP8%3D"
 			(at 96.52 90.17 90)
 			(effects
@@
 			)
 		)
-		(property "Sim.Name" ""
-			(at 96.52 90.17 90)
-			(effects
-				(font
-					(size 1.27 1.27)
-				)
-				(hide yes)
-			)
-		)
-		(property "Sim.Pins" ""
+		(property "Mouser No" "603-RT0603DRD0747RL"
 			(at 96.52 90.17 90)
 			(effects
@@
 			)
 		)
-		(property "Datasheet" "~"
+		(property "Datasheet" "https://www.mouser.pl/datasheet/3/508/1/PYu-RT_1-to-0.01_RoHS_L_15.pdf"
 			(at 96.52 100.33 0)
 			(effects
@@
 			)
 		)
-		(property "Sim.Device" ""
+		(property "Manufacturer_Part_Number" "RT0603DRD0747RL"
 			(at 96.52 100.33 90)
 			(effects
@@
 			)
 		)
-		(property "Sim.Library" ""
+		(property "Mouser" "https://www.mouser.pl/ProductDetail/YAGEO/RT0603DRD0747RL?qs=sGAEpiMZZMvdGkrng054t%252BSYh%252B1gqt95bcSQVS5MnP8%3D"
 			(at 96.52 100.33 90)
 			(effects
@@
 			)
 		)
-		(property "Sim.Name" ""
-			(at 96.52 100.33 90)
-			(effects
-				(font
-					(size 1.27 1.27)
-				)
-				(hide yes)
-			)
-		)
-		(property "Sim.Pins" ""
+		(property "Mouser No" "603-RT0603DRD0747RL"
 			(at 96.52 100.33 90)
 			(effects
@@
 			)
 		)
-		(property "Datasheet" "~"
+		(property "Datasheet" "https://www.mouser.pl/datasheet/3/508/1/PYu-RT_1-to-0.01_RoHS_L_15.pdf"
 			(at 175.26 78.74 0)
 			(effects
@@
 			)
 		)
-		(property "Sim.Device" ""
+		(property "Manufacturer_Part_Number" "RT0603DRD0747RL"
 			(at 175.26 78.74 90)
 			(effects
@@
 			)
 		)
-		(property "Sim.Library" ""
+		(property "Mouser" "https://www.mouser.pl/ProductDetail/YAGEO/RT0603DRD0747RL?qs=sGAEpiMZZMvdGkrng054t%252BSYh%252B1gqt95bcSQVS5MnP8%3D"
 			(at 175.26 78.74 90)
 			(effects
@@
 			)
 		)
-		(property "Sim.Name" ""
-			(at 175.26 78.74 90)
-			(effects
-				(font
-					(size 1.27 1.27)
-				)
-				(hide yes)
-			)
-		)
-		(property "Sim.Pins" ""
+		(property "Mouser No" "603-RT0603DRD0747RL"
 			(at 175.26 78.74 90)
 			(effects
@@
 			)
 		)
-		(property "Datasheet" "~"
+		(property "Datasheet" "https://www.mouser.pl/datasheet/3/508/1/PYu-RT_1-to-0.01_RoHS_L_15.pdf"
 			(at 175.26 88.9 0)
 			(effects
@@
 			)
 		)
-		(property "Sim.Device" ""
+		(property "Manufacturer_Part_Number" "RT0603DRD0747RL"
 			(at 175.26 88.9 90)
 			(effects
@@
 			)
 		)
-		(property "Sim.Library" ""
+		(property "Mouser" "https://www.mouser.pl/ProductDetail/YAGEO/RT0603DRD0747RL?qs=sGAEpiMZZMvdGkrng054t%252BSYh%252B1gqt95bcSQVS5MnP8%3D"
 			(at 175.26 88.9 90)
 			(effects
@@
 			)
 		)
-		(property "Sim.Name" ""
-			(at 175.26 88.9 90)
-			(effects
-				(font
-					(size 1.27 1.27)
-				)
-				(hide yes)
-			)
-		)
-		(property "Sim.Pins" ""
+		(property "Mouser No" "603-RT0603DRD0747RL"
 			(at 175.26 88.9 90)
 			(effects
@@
 			)
 		)
-		(property "Description" "STMicroelectronics Arm Cortex-M0+ MCU, 256KB flash, 144KB RAM, 64 MHz, 1.7-3.6V, 29 GPIO, LQFP32"
+		(property "Description" "MCU"
 			(at 133.35 92.71 0)
 			(effects
@@
 			)
 		)
-		(property "Sim.Device" ""
+		(property "Manufacturer_Part_Number" "STM32G0C1KCT6N"
 			(at 133.35 92.71 0)
 			(effects
@@
 			)
 		)
-		(property "Sim.Library" ""
+		(property "Mouser" "https://www.mouser.pl/ProductDetail/STMicroelectronics/STM32G0C1KCT6N?qs=iLbezkQI%252Bshu4f%252BBp0CpFw%3D%3D"
 			(at 133.35 92.71 0)
 			(effects
@@
 			)
 		)
-		(property "Sim.Name" ""
-			(at 133.35 92.71 0)
-			(effects
-				(font
-					(size 1.27 1.27)
-				)
-				(hide yes)
-			)
-		)
-		(property "Sim.Pins" ""
+		(property "Mouser No" "511-STM32G0C1KCT6N"
 			(at 133.35 92.71 0)
 			(effects
@@
 			)
 		)
-		(property "Datasheet" "~"
+		(property "Datasheet" "https://www.mouser.pl/datasheet/3/508/1/PYu-RT_1-to-0.01_RoHS_L_15.pdf"
 			(at 175.26 93.98 0)
 			(effects
@@
 			)
 		)
-		(property "Sim.Device" ""
+		(property "Manufacturer_Part_Number" "RT0603DRD0747RL"
 			(at 175.26 93.98 90)
 			(effects
@@
 			)
 		)
-		(property "Sim.Library" ""
+		(property "Mouser" "https://www.mouser.pl/ProductDetail/YAGEO/RT0603DRD0747RL?qs=sGAEpiMZZMvdGkrng054t%252BSYh%252B1gqt95bcSQVS5MnP8%3D"
 			(at 175.26 93.98 90)
 			(effects
@@
 			)
 		)
-		(property "Sim.Name" ""
-			(at 175.26 93.98 90)
-			(effects
-				(font
-					(size 1.27 1.27)
-				)
-				(hide yes)
-			)
-		)
-		(property "Sim.Pins" ""
+		(property "Mouser No" "603-RT0603DRD0747RL"
 			(at 175.26 93.98 90)
 			(effects
@@
 			)
 		)
-		(property "Datasheet" "~"
+		(property "Datasheet" "https://www.mouser.pl/datasheet/3/508/1/PYu-RT_1-to-0.01_RoHS_L_15.pdf"
 			(at 175.26 83.82 0)
 			(effects
@@
 			)
 		)
-		(property "Sim.Device" ""
+		(property "Manufacturer_Part_Number" "RT0603DRD0747RL"
 			(at 175.26 83.82 90)
 			(effects
@@
 			)
 		)
-		(property "Sim.Library" ""
+		(property "Mouser" "https://www.mouser.pl/ProductDetail/YAGEO/RT0603DRD0747RL?qs=sGAEpiMZZMvdGkrng054t%252BSYh%252B1gqt95bcSQVS5MnP8%3D"
 			(at 175.26 83.82 90)
 			(effects
@@
 			)
 		)
-		(property "Sim.Name" ""
+		(property "Mouser No" "603-RT0603DRD0747RL"
 			(at 175.26 83.82 90)
 			(effects
-				(font
-					(size 1.27 1.27)
-				)
-				(hide yes)
-			)
-		)
-		(property "Sim.Pins" ""
-			(at 175.26 83.82 90)
-			(effects
