File: hardware/Inputs.kicad_sch (KiCad schematic)
At the start: 52 parts, among them J13 Conn_01x05, J14 Conn_01x05, J15 Conn_01x05, J16 Conn_01x05, J17 Conn_01x05, J18 Conn_01x05, J19 Conn_01x03, J20 Conn_01x03, J21 Conn_01x03, J22 Conn_01x03, J23 Conn_01x03, J24 Conn_01x03, J25 Conn_01x02, J26 Conn_01x02, J27 FTSH-107-01-L-D-K

Commit message: Added all missing datasheet links etc
Parts:
- J13, J14, J15, J16, J17, J18: Manufacturer_Part_Number (none) -> 2601-1105; Mouser (none) -> https://www.wago.com/global/pcb-terminal-blocks-and-pluggab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; Mouser No (none) -> ---
- J19, J20, J21, J22, J23, J24: Manufacturer_Part_Number (none) -> 2601-1103; Mouser (none) -> https://www.wago.com/pl/złączki-do-płytek-drukowanych/złącz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; Mouser No (none) -> ---
- J25, J26: Manufacturer_Part_Number (none) -> strain relief; Mouser (none) -> ---
- J27: Manufacturer_Part_Nuber FTSH-107-01-L-D-K -> (none); Manufacturer_Part_Number (none) -> FTSH-107-01-L-D-K; Mouser No 200-FTSH10701LDK -> 200-FTSH10701LDK
- TP20, TP21, TP22, TP23, TP24, TP25, TP26, TP27, TP28, TP29, TP30, TP31, TP32, TP33, TP34, TP35, TP36, TP37: Manufacturer_Part_Number (none) -> ---; Mouser (none) -> ---; Mouser No (none) -> ---

Commit message: Corrections after review
Parts:
- J13, J14, J15, J16, J17, J18: Manufacturer_Part_Number 2601-1105 -> (none); Mouser https://www.wago.com/global/pcb-terminal-blocks-and-pluggab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 -> (none); Mouser No --- -> (none)
- J19, J20, J21, J22, J23, J24: Manufacturer_Part_Number 2601-1103 -> (none); Mouser https://www.wago.com/pl/złączki-do-płytek-drukowanych/złącz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 -> (none); Mouser No --- -> (none)
- J25, J26: Manufacturer_Part_Number strain relief -> (none); Mouser --- -> (none)
- J27: Manufacturer_Part_Nuber (none) -> FTSH-107-01-L-D-K; Manufacturer_Part_Number FTSH-107-01-L-D-K -> (none); Mouser No 200-FTSH10701LDK -> 200-FTSH10701LDK
- TP20, TP21, TP22, TP23, TP24, TP25, TP26, TP27, TP28, TP29, TP30, TP31, TP32, TP33, TP34, TP35, TP36, TP37: Manufacturer_Part_Number --- -> (none); Mouser --- -> (none); Mouser No --- -> (none)
