File: hardware/CAN.kicad_sch (KiCad schematic)
At the start: 15 parts, among them U3 ADM3057ExRW

Commit message: Corrections after review
Parts:
- R8: Manufacturer_Part_Number AC0603DR-07100KL -> (none); Mouser https://www.mouser.pl/ProductDetail/YAGEO/AC0603DR-07100KL?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 -> in warsztatowe zapasy i think; Mouser No 603-AC0603DR-07100KL -> (none)
Changed lines of the file:
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@@
 			)
 		)
-		(property "Mouser" "https://www.mouser.pl/ProductDetail/YAGEO/AC0603DR-07100KL?qs=sGAEpiMZZMvdGkrng054t3bQBroXiaAZB5Ggf8YdSs2QmcSO%2FG3V0Q%3D%3D"
+		(property "Mouser" "in warsztatowe zapasy i think"
 			(at 81.28 105.41 90)
 			(effects
-				(font
-					(size 1.27 1.27)
-				)
-				(hide yes)
-			)
-		)
-		(property "Manufacturer_Part_Number" "AC0603DR-07100KL"
-			(at 81.28 105.41 90)
-			(effects
-				(font
-					(size 1.27 1.27)
-				)
-				(hide yes)
-			)
-		)
-		(property "Mouser No" "603-AC0603DR-07100KL"
-			(at 81.28 105.41 90)
-			(effects

Commit message: Added Voltage reference, fixed silkscreen and BOM
Parts:
- R8: Manufacturer_Part_Number (none) -> RT0603FRE07174KL; Mouser in warsztatowe zapasy i think -> https://www.mouser.pl/ProductDetail/YAGEO/RT0603FRE07174KL?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; Mouser No (none) -> 603-RT0603FRE07174KL
Changed lines of the file:
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@@
 			)
 		)
-		(property "Mouser" "in warsztatowe zapasy i think"
+		(property "Mouser" "https://www.mouser.pl/ProductDetail/YAGEO/RT0603FRE07174KL?qs=4CyHz7GXqShAjm8rgsX%2FeQ%3D%3D"
 			(at 81.28 105.41 90)
 			(effects
+				(font
+					(size 1.27 1.27)
+				)
+				(hide yes)
+			)
+		)
+		(property "Manufacturer_Part_Number" "RT0603FRE07174KL"
+			(at 81.28 105.41 90)
+			(effects
+				(font
+					(size 1.27 1.27)
+				)
+				(hide yes)
+			)
+		)
+		(property "Mouser No" "603-RT0603FRE07174KL"
+			(at 81.28 105.41 90)
+			(effects
