File: hardware/CAN.kicad_sch (KiCad schematic)
At the start: 15 parts, among them U3 ADM3057ExRW

Commit message: Changed some components - they were non stocked
Parts:
- R8: Manufacturer_Part_Number RT0603FRE07174KL -> CRT0603-FZ-1003ELF; Mouser https://www.mouser.pl/ProductDetail/YAGEO/RT0603FRE07174KL?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 -> https://www.mouser.pl/ProductDetail/Bourns/CRT0603-FZ-1003E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; Mouser No 603-RT0603FRE07174KL -> 652-CRT0603FZ1003ELF
Changed lines of the file:
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@@
 			)
 		)
-		(property "Datasheet" "https://www.mouser.pl/datasheet/3/508/1/PYu-RT_1-to-0.01_RoHS_L_15.pdf"
+		(property "Datasheet" "https://www.mouser.pl/datasheet/3/40/1/CRT.pdf"
 			(at 81.28 105.41 0)
 			(effects
@@
 			)
 		)
-		(property "Mouser" "https://www.mouser.pl/ProductDetail/YAGEO/RT0603FRE07174KL?qs=4CyHz7GXqShAjm8rgsX%2FeQ%3D%3D"
+		(property "Mouser" "https://www.mouser.pl/ProductDetail/Bourns/CRT0603-FZ-1003ELF?qs=fgHA1UgJI8BbszSkndSeLg%3D%3D"
 			(at 81.28 105.41 90)
 			(effects
@@
 			)
 		)
-		(property "Manufacturer_Part_Number" "RT0603FRE07174KL"
+		(property "Manufacturer_Part_Number" "CRT0603-FZ-1003ELF"
 			(at 81.28 105.41 90)
 			(effects
@@
 			)
 		)
-		(property "Mouser No" "603-RT0603FRE07174KL"
+		(property "Mouser No" "652-CRT0603FZ1003ELF"
 			(at 81.28 105.41 90)
 			(effects
