File: hardware/CAN.kicad_sch (KiCad schematic)
At the start: 17 parts, among them U16 ADM3057EBRWZ

Commit message: style: fix board visuals
Parts:
- U16: footprint SOIC127P1032X265-20N -> ADM3057EBRWZ:SOIC127P1032X265-20N
Changed lines of the file:
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@@
 			)
 		)
-		(property "Footprint" "SOIC127P1032X265-20N"
+		(property "Footprint" "ADM3057EBRWZ:SOIC127P1032X265-20N"
 			(at 196.215 183.185 0)
 			(hide yes)
