File: hardware/UMB.kicad_pcb (KiCad board)
At the start: 6 copper layers, 128.8 x 67 mm, 213 parts, among them J1 PinHeader 02x04, J10 PH1-03-UA, J11 PH1-03-UA, J12 PH1-03-UA, J13 Conn_01x05, J14 Conn_01x05, J15 Conn_01x05, J16 Conn_01x05, J17 Conn_01x05, J18 Conn_01x05, J19 Conn_01x03, J2 PinHeader 02x04, J20 Conn_01x03, J21 Conn_01x03, J22 Conn_01x03, J23 Conn_01x03, J24 Conn_01x03, J25 Conn_01x02, J26 Conn_01x02, J27 FTSH-107-01-L-D-K, J3 PinHeader 02x04, J4 PinHeader 02x04, J5 PinHeader 02x04, J6 PinHeader 02x04, J7 PH1-03-UA, J8 PH1-03-UA, J9 PH1-03-UA, U1 STM32G0C1KCTxN, U10 LDK320ADU120R, U11 INA2128UA_1K, U12 INA2128UA_1K, U13 INA2128UA_1K, U14 TLC274AIDR, U15 TLC274AIDR, U16 TLC274AIDR, U2 ADS114S08BIPBSR, U3 ADM3057ExRW, U4 TPS563300DRLR, U5 TPS563219ADDFR, U6 LM2940SX-12_NOPB, U7 LM1117IMP-5.0, U8 TLV743P, U9 AP2127N3-1.5

Commit message: Added Voltage reference, fixed silkscreen and BOM
Parts:
- removed the ? at (97.9, 107.4)
- added R56: 2.1k, Resistor_SMD:R_0603_1608Metric_Pad0.98x0.95mm_HandSolder, F.Cu at (102.0, 107.0)
- added R57: 10k, Resistor_SMD:R_0603_1608Metric_Pad0.98x0.95mm_HandSolder, F.Cu at (99.5, 109.2)
- added R58: 10k, Resistor_SMD:R_0603_1608Metric_Pad0.98x0.95mm_HandSolder, F.Cu at (98.5, 111.8)
- added U17: TL431LIBQDBZRQ1, Package_TO_SOT_SMD:SOT-23W_Handsoldering, F.Cu at (102.0, 110.8)
- moved ? 1.03 mm to (117.4, 106.5)
- renumbered 20 to TP20, 21 to TP21, 22 to TP22, 23 to TP23, 24 to TP24, 25 to TP25, 26 to TP26, 27 to TP27, 28 to TP28, 29 to TP29, 30 to TP30, 31 to TP31, 34 to TP34, 37 to TP37, 9 to TP9
Connections:
- U11 pad 12: GND -> +6VA
- U11 pad 5: GND -> +6VA
- U12 pad 12: GND -> +6VA
- U12 pad 5: GND -> +6VA
- U13 pad 12: GND -> +6VA
- U13 pad 5: GND -> +6VA
Routing:
- net +6VA: track 0.00 -> 116.2 mm, vias 0 -> 7
- net GND: track 197.1 -> 190.7 mm, vias 168 -> 164
- net Net-(U17-REF): track 0.00 -> 4.02 mm
- net Net-(U14B--): track 26.2 -> 25.2 mm
- net +5VA: vias 31 -> 32
- net +12VA: vias 7 -> 5

Commit message: Fixed R57 value
Parts:
- R57: value 10k -> 14k
