File: hardware/ADC.kicad_sch (KiCad schematic)
At the start: 4 parts, among them U2 ADS114S08BIPBSR

Commit message: hardware sync
Parts:
- added C44: 1u, Capacitor_SMD:C_0603_1608Metric_Pad1.08x0.95mm_HandSolder, symbol Device:C_Small
Connections:
- net +5VA: now also U2.30 (REFP0), C44.1
- net GND: now also U2.1 (AINCOM), U2.29 (REFN0), C44.2
- no-connect marks 3 -> 0
Other:
- moved on the sheet: C3
