File: hardware/Connectors.kicad_sch (KiCad schematic)
At the start: 44 parts, among them J1 2606-1110_010-000, J2 2606-1110_010-000, J3 2606-1110_010-000, J4 2606-1110_010-000, J5 Strain Relief, J6 Strain Relief, J7 FTSH-107-01-L-D-K, J8 Strain Relief, J9 Strain Relief

Commit message: style: fix board visuals
Parts:
- D10, D11, D12, D13, D14, D15, D16, D17, D18, D3, D4, D5, D6, D7, D8, D9: footprint SODFL3718X130N -> ATV02W150-HF:SODFL3718X130N
- D19: footprint SOT95P230X110-3N -> PESD5V0L2BT,215:SOT95P230X110-3N
- D20, D21: footprint SOT95P280X145-5N -> ESDS304DBVR:SOT95P280X145-5N
Changed lines of the file:
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@@
 		(fields_autoplaced yes)
 		(property "Reference" "D21"
-			(at 86.995 205.105 0)
+			(at 86.995 204.47 0)
 			(show_name no)
 			(do_not_autoplace no)
@@
 		)
 		(property "Value" "ESDS304DBVR"
-			(at 86.995 207.645 0)
+			(at 86.995 207.01 0)
 			(show_name no)
 			(do_not_autoplace no)
@@
 			)
 		)
-		(property "Footprint" "SOT95P280X145-5N"
+		(property "Footprint" "ESDS304DBVR:SOT95P280X145-5N"
 			(at 111.125 305.74 0)
 			(hide yes)
@@
 		(fields_autoplaced yes)
 		(property "Reference" "D18"
-			(at 313.055 125.7299 90)
+			(at 312.42 125.7299 90)
 			(show_name no)
 			(do_not_autoplace no)
@@
 		)
 		(property "Value" "ATV02W150-HF"
-			(at 313.055 128.2699 90)
+			(at 312.42 128.2699 90)
 			(show_name no)
 			(do_not_autoplace no)
@@
 			)
 		)
-		(property "Footprint" "SODFL3718X130N"
+		(property "Footprint" "ATV02W150-HF:SODFL3718X130N"
 			(at 403.53 116.84 0)
 			(hide yes)
@@
 			)
 		)
-		(property "Footprint" "SODFL3718X130N"
+		(property "Footprint" "ATV02W150-HF:SODFL3718X130N"
 			(at 380.035 67.945 0)
 			(hide yes)
@@
 			)
 		)
-		(property "Footprint" "SOT95P280X145-5N"
+		(property "Footprint" "ESDS304DBVR:SOT95P280X145-5N"
 			(at 139.065 315.265 0)
 			(hide yes)
@@
 			)
 		)
-		(property "Footprint" "SODFL3718X130N"
+		(property "Footprint" "ATV02W150-HF:SODFL3718X130N"
 			(at 199.695 116.84 0)
 			(hide yes)
@@
 			)
 		)
-		(property "Footprint" "SODFL3718X130N"
+		(property "Footprint" "ATV02W150-HF:SODFL3718X130N"
 			(at 176.2 67.945 0)
 			(hide yes)
@@
 			)
 		)
-		(property "Footprint" "SODFL3718X130N"
+		(property "Footprint" "ATV02W150-HF:SODFL3718X130N"
 			(at 176.2 114.935 0)
 			(hide yes)
@@
 			)
 		)
-		(property "Footprint" "SOT95P280X145-5N"
+		(property "Footprint" "ESDS304DBVR:SOT95P280X145-5N"
 			(at 139.065 295.58 0)
 			(hide yes)
@@
 			)
 		)
-		(property "Footprint" "SOT95P280X145-5N"
+		(property "Footprint" "ESDS304DBVR:SOT95P280X145-5N"
 			(at 139.065 305.74 0)
 			(hide yes)
@@
 			)
 		)
-		(property "Footprint" "SODFL3718X130N"
+		(property "Footprint" "ATV02W150-HF:SODFL3718X130N"
 			(at 335.585 69.85 0)
 			(hide yes)
@@
 			)
 		)
-		(property "Footprint" "SODFL3718X130N"
+		(property "Footprint" "ATV02W150-HF:SODFL3718X130N"
 			(at 244.145 67.945 0)
 			(hide yes)
@@
 			)
 		)
-		(property "Footprint" "SODFL3718X130N"
+		(property "Footprint" "ATV02W150-HF:SODFL3718X130N"
 			(at 244.145 114.935 0)
 			(hide yes)
@@
 			)
 		)
-		(property "Footprint" "SOT95P280X145-5N"
+		(property "Footprint" "ESDS304DBVR:SOT95P280X145-5N"
 			(at 111.125 315.265 0)
 			(hide yes)
@@
 		(fields_autoplaced yes)
 		(property "Reference" "D19"
-			(at 196.215 186.6899 90)
+			(at 196.85 186.6899 90)
 			(show_name no)
 			(do_not_autoplace no)
@@
 		)
 		(property "Value" "PESD5V0L2BT,215"
-			(at 196.215 189.2299 90)
+			(at 196.85 189.2299 90)
 			(show_name no)
 			(do_not_autoplace no)
@@
 			)
 		)
-		(property "Footprint" "SOT95P230X110-3N"
+		(property "Footprint" "PESD5V0L2BT,215:SOT95P230X110-3N"
 			(at 114.63 214.63 0)
 			(hide yes)
@@
 			)
 		)
-		(property "Footprint" "SODFL3718X130N"
+		(property "Footprint" "ATV02W150-HF:SODFL3718X130N"
 			(at 312.09 114.935 0)
 			(hide yes)
@@
 			)
 		)
-		(property "Footprint" "SOT95P280X145-5N"
+		(property "Footprint" "ESDS304DBVR:SOT95P280X145-5N"
 			(at 111.125 295.58 0)
 			(hide yes)
@@
 			)
 		)
-		(property "Footprint" "SOT95P280X145-5N"
+		(property "Footprint" "ESDS304DBVR:SOT95P280X145-5N"
 			(at 111.125 325.425 0)
 			(hide yes)
@@
 			)
 		)
-		(property "Footprint" "SODFL3718X130N"
+		(property "Footprint" "ATV02W150-HF:SODFL3718X130N"
 			(at 199.695 69.85 0)
 			(hide yes)
@@
 			)
 		)
-		(property "Footprint" "SOT95P230X110-3N"
+		(property "Footprint" "PESD5V0L2BT,215:SOT95P230X110-3N"
 			(at 89.865 211.455 0)
 			(hide yes)
@@
 			)
 		)
-		(property "Footprint" "SODFL3718X130N"
+		(property "Footprint" "ATV02W150-HF:SODFL3718X130N"
 			(at 267.64 69.85 0)
 			(hide yes)
@@
 			)
 		)
-		(property "Footprint" "SODFL3718X130N"
+		(property "Footprint" "ATV02W150-HF:SODFL3718X130N"
 			(at 267.64 116.84 0)
 			(hide yes)
@@
 			)
 		)
-		(property "Footprint" "SOT95P280X145-5N"
+		(property "Footprint" "ESDS304DBVR:SOT95P280X145-5N"
 			(at 139.065 325.425 0)
 			(hide yes)
@@
 		(fields_autoplaced yes)
 		(property "Reference" "D10"
-			(at 313.055 78.7399 90)
+			(at 312.42 78.7399 90)
 			(show_name no)
 			(do_not_autoplace no)
@@
 		)
 		(property "Value" "ATV02W150-HF"
-			(at 313.055 81.2799 90)
+			(at 312.42 81.2799 90)
 			(show_name no)
 			(do_not_autoplace no)
@@
 			)
 		)
-		(property "Footprint" "SODFL3718X130N"
+		(property "Footprint" "ATV02W150-HF:SODFL3718X130N"
 			(at 403.53 69.85 0)
 			(hide yes)
@@
 			)
 		)
-		(property "Footprint" "SODFL3718X130N"
+		(property "Footprint" "ATV02W150-HF:SODFL3718X130N"
 			(at 312.09 67.945 0)
 			(hide yes)
@@
 			)
 		)
-		(property "Footprint" "SODFL3718X130N"
+		(property "Footprint" "ATV02W150-HF:SODFL3718X130N"
 			(at 335.585 116.84 0)
 			(hide yes)
@@
 			)
 		)
-		(property "Footprint" "SODFL3718X130N"
+		(property "Footprint" "ATV02W150-HF:SODFL3718X130N"
 			(at 380.035 114.935 0)
 			(hide yes)
