File: hardware/Conv.kicad_sch (KiCad schematic)
At the start: 101 parts, among them U10 LT3471EDD#PBF, U11 L7812ABD2T-TR, U12 ISL21010CFH330Z-TK, U13 L78L15ACD13TR, U14 TPS54202HDDCR, U15 L79L15ACD13TR, U5 UA78M33CDCYRG3, U6 TPS54202HDDCR, U7 UA78M33CDCYRG3, U8 L7805ABD2T-TR, U9 ISL21010CFH315Z-TK

Commit message: style: fix board visuals
Parts:
- L1: footprint 74437349560 -> 74437349560:74437349560
- U10: footprint SON50P300X300X80-11N-D -> LT3471EDD#PBF:SON50P300X300X80-11N-D
- U11, U8: footprint L7805ABD2TTR -> L7805ABD2T-TR:L7805ABD2TTR
- U12, U9: footprint SOT95P237X112-3N -> ISL21010CFH315Z-TK:SOT95P237X112-3N
- U13: footprint SOIC127P600X175-8N -> L78L15ACD13TR:SOIC127P600X175-8N
- U14, U6: footprint SOT95P280X110-6N -> TPS54202HDDCR:SOT95P280X110-6N
- U15: footprint SOIC127P600X175-8N -> L79L15ACD13TR:SOIC127P600X175-8N
- U5, U7: footprint SOT230P700X180-4N -> UA78M33CDCYRG3:SOT230P700X180-4N
Changed lines of the file:
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@@
 			)
 		)
-		(property "Footprint" "L7805ABD2TTR"
+		(property "Footprint" "L7805ABD2T-TR:L7805ABD2TTR"
 			(at 265.43 232.08 0)
 			(hide yes)
@@
 		(fields_autoplaced yes)
 		(property "Reference" "U14"
-			(at 112.395 167.005 0)
+			(at 112.395 167.64 0)
 			(show_name no)
 			(do_not_autoplace no)
@@
 		)
 		(property "Value" "TPS54202HDDCR"
-			(at 112.395 169.545 0)
+			(at 112.395 170.18 0)
 			(show_name no)
 			(do_not_autoplace no)
@@
 			)
 		)
-		(property "Footprint" "SOT95P280X110-6N"
+		(property "Footprint" "TPS54202HDDCR:SOT95P280X110-6N"
 			(at 136.525 277.165 0)
 			(hide yes)
@@
 			)
 		)
-		(property "Footprint" "SON50P300X300X80-11N-D"
+		(property "Footprint" "LT3471EDD#PBF:SON50P300X300X80-11N-D"
 			(at 152.4 203.505 0)
 			(hide yes)
@@
 		(fields_autoplaced yes)
 		(property "Reference" "U9"
-			(at 316.865 104.775 0)
+			(at 316.865 105.41 0)
 			(show_name no)
 			(do_not_autoplace no)
@@
 		)
 		(property "Value" "ISL21010CFH315Z-TK"
-			(at 316.865 107.315 0)
+			(at 316.865 107.95 0)
 			(show_name no)
 			(do_not_autoplace no)
@@
 			)
 		)
-		(property "Footprint" "SOT95P237X112-3N"
+		(property "Footprint" "ISL21010CFH315Z-TK:SOT95P237X112-3N"
 			(at 340.995 211.125 0)
 			(hide yes)
@@
 		(fields_autoplaced yes)
 		(property "Reference" "U8"
-			(at 233.68 97.155 0)
+			(at 233.68 96.52 0)
 			(show_name no)
 			(do_not_autoplace no)
@@
 		)
 		(property "Value" "L7805ABD2T-TR"
-			(at 233.68 99.695 0)
+			(at 233.68 99.06 0)
 			(show_name no)
 			(do_not_autoplace no)
@@
 			)
 		)
-		(property "Footprint" "L7805ABD2TTR"
+		(property "Footprint" "L7805ABD2T-TR:L7805ABD2TTR"
 			(at 260.35 200.33 0)
 			(hide yes)
@@
 			)
 		)
-		(property "Footprint" "SOT230P700X180-4N"
+		(property "Footprint" "UA78M33CDCYRG3:SOT230P700X180-4N"
 			(at 267.97 136.83 0)
 			(hide yes)
@@
 		(fields_autoplaced yes)
 		(property "Reference" "U13"
-			(at 233.68 160.655 0)
+			(at 233.68 160.02 0)
 			(show_name no)
 			(do_not_autoplace no)
@@
 		)
 		(property "Value" "L78L15ACD13TR"
-			(at 233.68 163.195 0)
+			(at 233.68 162.56 0)
 			(show_name no)
 			(do_not_autoplace no)
@@
 			)
 		)
-		(property "Footprint" "SOIC127P600X175-8N"
+		(property "Footprint" "L78L15ACD13TR:SOIC127P600X175-8N"
 			(at 260.35 263.83 0)
 			(hide yes)
@@
 			)
 		)
-		(property "Footprint" "SOT95P280X110-6N"
+		(property "Footprint" "TPS54202HDDCR:SOT95P280X110-6N"
 			(at 129.54 143.18 0)
 			(hide yes)
@@
 		(fields_autoplaced yes)
 		(property "Reference" "L1"
-			(at 123.825 34.925 0)
+			(at 123.825 35.56 0)
 			(show_name no)
 			(do_not_autoplace no)
@@
 		)
 		(property "Value" "74437349560"
-			(at 123.825 37.465 0)
+			(at 123.825 38.1 0)
 			(show_name no)
 			(do_not_autoplace no)
@@
 			)
 		)
-		(property "Footprint" "74437349560"
+		(property "Footprint" "74437349560:74437349560"
 			(at 140.335 136.83 0)
 			(hide yes)
@@
 			)
 		)
-		(property "Footprint" "SOIC127P600X175-8N"
+		(property "Footprint" "L79L15ACD13TR:SOIC127P600X175-8N"
 			(at 260.35 100.025 0)
 			(hide yes)
@@
 			)
 		)
-		(property "Footprint" "SOT95P237X112-3N"
+		(property "Footprint" "ISL21010CFH315Z-TK:SOT95P237X112-3N"
 			(at 340.995 241.605 0)
 			(hide yes)
@@
 			)
 		)
-		(property "Footprint" "SOT230P700X180-4N"
+		(property "Footprint" "UA78M33CDCYRG3:SOT230P700X180-4N"
 			(at 267.97 168.58 0)
 			(hide yes)
