File: hardware/MCU.kicad_sch (KiCad schematic)
At the start: 14 parts, among them U1 ADS8863IDGS, U2 STM32G484RET3, Y1 ATX-H11-F-16.000MHz-G100-T

Commit message: style: fix board visuals
Parts:
- U1: footprint SOP50P490X110-10N -> ADS8863IDGS:SOP50P490X110-10N
- U2: footprint QFP50P1200X1200X160-64N -> STM32G484RET3:QFP50P1200X1200X160-64N
- Y1: footprint ATXH11F16000MHzG100T -> ATX-H11-F-16.000MHz-G100-T:ATXH11F16000MHzG100T
Changed lines of the file:
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@@
 		(fields_autoplaced yes)
 		(property "Reference" "Y1"
-			(at 198.12 107.315 0)
+			(at 198.12 107.95 0)
 			(show_name no)
 			(do_not_autoplace no)
@@
 		)
 		(property "Value" "ATX-H11-F-16.000MHz-G100-T"
-			(at 198.12 109.855 0)
-			(show_name no)
-			(do_not_autoplace no)
-			(effects
-				(font
-					(size 1.27 1.27)
-				)
-			)
-		)
-		(property "Footprint" "ATXH11F16000MHzG100T"
+			(at 198.12 110.49 0)
+			(show_name no)
+			(do_not_autoplace no)
+			(effects
+				(font
+					(size 1.27 1.27)
+				)
+			)
+		)
+		(property "Footprint" "ATX-H11-F-16.000MHz-G100-T:ATXH11F16000MHzG100T"
 			(at 224.79 212.395 0)
 			(hide yes)
@@
 			)
 		)
-		(property "Footprint" "QFP50P1200X1200X160-64N"
+		(property "Footprint" "STM32G484RET3:QFP50P1200X1200X160-64N"
 			(at 158.75 177.47 0)
 			(hide yes)
@@
 		(fields_autoplaced yes)
 		(property "Reference" "U1"
-			(at 233.68 43.815 0)
+			(at 233.68 44.45 0)
 			(show_name no)
 			(do_not_autoplace no)
@@
 		)
 		(property "Value" "ADS8863IDGS"
-			(at 233.68 46.355 0)
-			(show_name no)
-			(do_not_autoplace no)
-			(effects
-				(font
-					(size 1.27 1.27)
-				)
-			)
-		)
-		(property "Footprint" "SOP50P490X110-10N"
+			(at 233.68 46.99 0)
+			(show_name no)
+			(do_not_autoplace no)
+			(effects
+				(font
+					(size 1.27 1.27)
+				)
+			)
+		)
+		(property "Footprint" "ADS8863IDGS:SOP50P490X110-10N"
 			(at 232.41 134.925 0)
 			(hide yes)
