File: hardware/UNIVERSAL_MEASURMENT_BOARD.kicad_pcb (KiCad board)
At the start: 6 copper layers, 75 x 95 mm, 177 parts, among them J1 2606-1110_010-000, J2 2606-1110_010-000, J3 2606-1110_010-000, J4 2606-1110_010-000, J5 Strain Relief, J6 Strain Relief, J7 FTSH-107-01-L-D-K, J8 Strain Relief, J9 Strain Relief, U1 ADS8863IDGS, U10 LT3471EDD#PBF, U11 L7812ABD2T-TR, U12 ISL21010CFH330Z-TK, U13 L78L15ACD13TR, U14 TPS54202HDDCR, U15 L79L15ACD13TR, U16 ADM3057EBRWZ, U2 STM32G484RET3, U3 PGA280AIPW, U4 CD4097BM, U5 UA78M33CDCYRG3, U6 TPS54202HDDCR, U7 UA78M33CDCYRG3, U8 L7805ABD2T-TR, U9 ISL21010CFH315Z-TK, Y1 ATX-H11-F-16.000MHz-G100-T

Commit message: style: fix board visuals
Parts:
- added REF**: Screw_Generic_2.0x3.0mm_SilkScreen, Symbol:Screw_Generic_2.0x3.0mm_SilkScreen, F.Cu at (109.3, 128.9)
- added REF**: Screw_Generic_2.0x3.0mm_SilkScreen, Symbol:Screw_Generic_2.0x3.0mm_SilkScreen, B.Cu at (39.8, 52.9)
- added REF**: Screw_Generic_2.0x3.0mm_SilkScreen, Symbol:Screw_Generic_2.0x3.0mm_SilkScreen, B.Cu at (109.3, 53.4)
- added REF**: Screw_Generic_2.0x3.0mm_SilkScreen, Symbol:Screw_Generic_2.0x3.0mm_SilkScreen, B.Cu at (39.8, 128.3)
- added REF**: Screw_Generic_2.0x3.0mm_SilkScreen, Symbol:Screw_Generic_2.0x3.0mm_SilkScreen, F.Cu at (39.8, 52.9)
- added REF**: Screw_Generic_2.0x3.0mm_SilkScreen, Symbol:Screw_Generic_2.0x3.0mm_SilkScreen, F.Cu at (39.8, 128.9)
- added REF**: Screw_Generic_2.0x3.0mm_SilkScreen, Symbol:Screw_Generic_2.0x3.0mm_SilkScreen, F.Cu at (109.3, 52.9)
- added REF**: Screw_Generic_2.0x3.0mm_SilkScreen, Symbol:Screw_Generic_2.0x3.0mm_SilkScreen, B.Cu at (109.3, 128.9)
- U13: footprint LP358DR:SOIC127P600X175-8N -> L78L15ACD13TR:SOIC127P600X175-8N
- U15: footprint LP358DR:SOIC127P600X175-8N -> L79L15ACD13TR:SOIC127P600X175-8N
- turned U13 to 0 degrees
- turned U15 to 0 degrees
Connections:
- REF** pad 1: (no net) -> GND (x4)
Other:
- board text added: "A: Marcin Trzmiel R: Piotr Witt R: Grzegorz Potocki"
- board text added: "Uniwersal Measurement Board Dat.: 28.06.2026 Rev.: 2.0"
- board text removed: "A: Marcin Trzmiel R: Piotr Lesicki R: Piotr Witt"
- board text removed: "Uniwersal Measurement Board Dat.: Rev.: 2.0"
