File: hardware/mux & pga.kicad_sch (KiCad schematic)
At the start: 11 parts, among them U3 PGA280AIPW, U4 CD4097BM

Commit message: style: fix board visuals
Parts:
- U4: footprint SOIC127P1030X265-24N -> CD4097BM:SOIC127P1030X265-24N
Changed lines of the file:
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@@
 		(fields_autoplaced yes)
 		(property "Reference" "U4"
-			(at 57.785 126.365 0)
+			(at 57.785 127 0)
 			(show_name no)
 			(do_not_autoplace no)
@@
 		)
 		(property "Value" "CD4097BM"
-			(at 57.785 128.905 0)
+			(at 57.785 129.54 0)
 			(show_name no)
 			(do_not_autoplace no)
@@
 			)
 		)
-		(property "Footprint" "SOIC127P1030X265-24N"
+		(property "Footprint" "CD4097BM:SOIC127P1030X265-24N"
 			(at 112.395 259.385 0)
 			(hide yes)
