File: hardware/UNIVERSAL_MEASURMENT_BOARD/UNIVERSAL_MEASURMENT_BOARD.kicad_pcb (KiCad board)
At the start: 6 copper layers, 70 x 135 mm, 191 parts, among them J1 FTSH-107-01-L-D-K, J2 2606-1110_010-000, J3 2606-1110_010-000, J4 Conn_01x01_Socket, J5 Conn_01x01_Socket, J6 Conn_01x01_Socket, J7 Conn_01x01_Socket, J8 2606-1110_010-000, J9 2606-1110_010-000, U1 STM32G484RET3, U10 L7805ABD2T-TR, U11 L7812ABD2T-TR, U12 L78L15ACD13TR, U13 L79L15ACD13TR, U14 ISL21010CFH315Z-TK, U15 ISL21010CFH330Z-TK, U16 ESDS304DBVR, U17 ESDS304DBVR, U18 ADM3055EBRIZ-RL, U2 ADS8863IDGS, U3 PGA280AIPW, U4 CD4097BM, U5 TPS54202HDDCR, U6 TPS54202HDDCR, U7 LT3471EDD#PBF, U8 UA78M33CDCYRG3, U9 UA78M33CDCYRG3, Y1 ECS-1612MV

Commit message: Review fixes
Parts:
- added C80: 10uF, REST:C_0805_2012Metric, F.Cu at (116.7, 68.9)
- J4, J5, J6, J7: footprint REST:SolderWire-0.1sqmm_1x01_D0.4mm_OD1mm_Relief2x -> REST:SolderPoint
- U18: value ADM3055EBRIZ-RL -> ADM3057EBRWZ; footprint ADM3055EBRIZ-RL:SOIC127P1030X264-20N -> ADM3057EBRWZ:SOIC127P1032X265-20N
- Y1: value ECS-1612MV -> ATX-H11-F-16.000MHz-G100-T; footprint ECS-1612MV-080-CN-TR:ECS1612MV080CNTR -> ATX-H11-F-16.000MHz-G100-T:ATXH11F16000MHzG100T
- moved C11 42.7 mm to (100.9, 140.1)
- moved D2 38.2 mm to (123.1, 54.9), turned to 180 degrees
- moved C27 33.3 mm to (109.1, 70.0)
- moved C8 33.2 mm to (87.9, 132.1)
- moved R2 32.6 mm to (87.9, 130.5)
- moved TP2 32.2 mm to (127.1, 64.1)
- moved J1 32.1 mm to (94.4, 87.9), turned to 180 degrees
- moved C31 31.5 mm to (111.0, 55.1), turned to 180 degrees
- moved C30 30.3 mm to (127.1, 65.1), turned to 90 degrees
- moved R13 30.1 mm to (109.1, 66.9)
- moved C24 29.9 mm to (115.2, 57.1), turned to -135 degrees
- moved D3 29.7 mm to (82.8, 94.3)
- moved D5 29.7 mm to (82.8, 97.8)
- moved F4 29.7 mm to (82.8, 87.3)
- moved F5 29.7 mm to (82.8, 90.8)
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Connections:
- L1 pad 1: +15V0F -> Net-(U7-SW2)
- L1 pad 2: Net-(U7-SW2) -> +15V0F
- U1 pad 11: /mcu & adc/ADDR2 -> unconnected-(U1-PC3-Pad11)
- U1 pad 12: /mcu & adc/ADDR1 -> unconnected-(U1-PA0-Pad12)
- U1 pad 13: /mcu & adc/MUXEN -> unconnected-(U1-PA1-Pad13)
- U1 pad 14: /mcu & adc/ADDR3 -> unconnected-(U1-PA2-Pad14)
- U1 pad 18: unconnected-(U1-PA4-Pad18) -> /mcu & adc/ADCCS
- U1 pad 22: /mcu & adc/ADCCS -> unconnected-(U1-PC4-Pad22)
- U1 pad 33: unconnected-(U1-PB11-Pad33) -> /mcu & adc/ADDR1
- U1 pad 34: unconnected-(U1-PB12-Pad34) -> /mcu & adc/ADDR2
- U1 pad 35: unconnected-(U1-PB13-Pad35) -> /mcu & adc/MUXEN
- U1 pad 36: unconnected-(U1-PB14-Pad36) -> /mcu & adc/ADDR3
- U16 pad 1: unconnected-(U16-Pad1) -> /connectors/NRST
- U16 pad 3: /connectors/SWDIO -> /connectors/UART_TX_PROG
- U16 pad 4: /connectors/SWCLK -> /connectors/UART_RX_PROG
- U16 pad 5: /connectors/SWO -> +3V3
- U17 pad 1: /connectors/UART_RX_PROG -> /connectors/SWCLK
- U17 pad 3: unconnected-(U17-Pad3) -> /connectors/SWDIO
- U17 pad 4: /connectors/NRST -> GND
- U17 pad 5: /connectors/UART_TX_PROG -> /connectors/SWO
- Y1 pad 1: GND -> +3V3
Routing:
- net /connectors/A1N: track 84.5 -> 139.4 mm
- net /connectors/A8P: track 94.3 -> 144.2 mm, vias 2 -> 3
- net /connectors/A2N: track 71.8 -> 117.2 mm
- net +5V0A: track 254.7 -> 299.7 mm, vias 15 -> 12
- net /connectors/A7P: track 81.9 -> 121.0 mm, vias 2 -> 3
- net +12V0A: track 202.4 -> 236.1 mm, vias 7 -> 21
- net /connectors/A3N: track 57.8 -> 90.8 mm
- net +7V0: track 33.1 -> 1.84 mm, vias 41 -> 23
- net /connectors/A6P: track 67.6 -> 96.8 mm, vias 2 -> 3
- net +15V0F: track 5.17 -> 32.7 mm, vias 14 -> 13
- net /connectors/SWDIO: track 36.1 -> 11.7 mm, vias 2 -> 0
- net -18V0: track 29.9 -> 53.1 mm, vias 24 -> 13
- net /connectors/A4N: track 45.0 -> 67.9 mm
- net +3V0A: track 57.9 -> 80.6 mm, vias 5 -> 4
- net +18V0: track 61.5 -> 41.8 mm
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- added copper zone on B.Cu, net +7V0
- added copper zone on B.Cu, net GND
- added copper zone on In2.Cu, net GND
- added copper zone on In3.Cu, net GND
- added copper zone on F.Cu, net GND_ISO
- removed copper zone on F.Cu, net Net-(U5-BOOT)
- removed copper zone on F.Cu, net Net-(U5-SW)
- removed copper zone on B.Cu, net Net-(U5-VIN)
- removed copper zone on F.Cu, net Net-(U6-SW)
Other:
- board text added: "L6"
- board text added: "STACKUP: 1. SIGNAL / POWER 2. GND 3. SIGNAL / POWER ON PS 4. SIGNAL / POWER ON PS 5. GND 6. SIGNAL / POWER"
- board text removed: "STACKUP: 1. SIGNAL / POWER 2. GND 3. SIGNAL 4. SIGNAL 5. GND 6. SIGNAL / POWER"

Commit message: Additional review fixes
Routing:
- net -18V0: track 53.1 -> 30.2 mm
- net +3V3: track 234.9 -> 247.1 mm
- net GND: vias 898 -> 835
- net +5V0A: vias 12 -> 11
Other:
- board text added: "A: Marcin Trzmiel R: Piotr Lesicki R: Piotr Witt"
- board text added: "Uniwersal Measurement Board Rev.: 1.0"
- board text removed: "Marcin Trzmiel"
- board text removed: "Measurement Board Rev.: 1.0"
